File: UccMicroDuino/UccMicroDuino.kicad_pcb (KiCad board)
At the start: 2 copper layers, 8 parts, among them J1 Conn_01x10_Socket, J2 USB_A, U1 ATtiny85-20S

Commit message: Comienzo de cableado
Parts:
- added D3: 3.6V 1/2mW, Diode_SMD:D_SOD-123, F.Cu at (197.3, 86.5)
- added D4: LED Green, ledSmd:ledSMD, F.Cu at (211.0, 102.5)
- added R2: 68Ω 5% 1/8w, Resistor_SMD:R_0805_2012Metric_Pad1.20x1.40mm_HandSolder, F.Cu at (205.5, 76.0)
- added R3: 68Ω 5% 1/8w, Resistor_SMD:R_0805_2012Metric_Pad1.20x1.40mm_HandSolder, F.Cu at (205.5, 79.0)
- added R4: 330Ω 5% 1/8w, Resistor_SMD:R_0805_2012Metric_Pad1.20x1.40mm_HandSolder, F.Cu at (195.2, 98.5)
- added R5: 330Ω 5% 1/8w, Resistor_SMD:R_0805_2012Metric_Pad1.20x1.40mm_HandSolder, F.Cu at (222.5, 70.0)
- C1: value C -> 0.1u
- D1: value D_Filled -> PMLL4148L
- D2: value D_Zener -> 3.6V 1/2mW
- D5: renamed from D3; value LED -> LED Red
- J1: renamed from J2; value USB_A -> Pcb USB type A
- J2: renamed from J1; value Conn_01x10_Socket -> Header
- R1: value R -> 1.5 kΩ 5% 1/8w
- U1: footprint Package_SO:SOIC-8W_5.3x5.3mm_P1.27mm -> Package_SO:SOIC-8_5.3x5.3mm_P1.27mm
- moved D5 87.4 mm to (222.5, 76.5), turned to -90 degrees
- moved U1 87.2 mm to (218.3, 92.2)
- moved J2 87.0 mm to (200.7, 109.2), turned to 90 degrees
- moved C1 71.5 mm to (195.5, 110.5)
- moved D2 69.1 mm to (197.8, 81.3)
- moved D1 69.0 mm to (196.2, 105.3)
- moved R1 64.9 mm to (203.5, 70.5)
- moved J1 54.2 mm to (186.2, 73.5)
Connections:
- C1 pad 1: unconnected-(C1-Pad1) -> +5V
- C1 pad 2: unconnected-(C1-Pad2) -> (no net)
- D1 pad 2: unconnected-(D1-A-Pad2) -> (no net)
- D2 pad 1: unconnected-(D2-K-Pad1) -> (no net)
- D2 pad 2: unconnected-(D2-A-Pad2) -> GND
- D5 pad 1: unconnected-(D3-K-Pad1) -> (no net)
- D5 pad 2: unconnected-(D3-A-Pad2) -> +5V
- J1 pad 1: unconnected-(J2-VBUS-Pad1) -> Net-(D1-A)
- J1 pad 2: unconnected-(J2-D--Pad2) -> Net-(D2-K)
- J1 pad 3: unconnected-(J2-D+-Pad3) -> Net-(D3-K)
- J1 pad 4: unconnected-(J2-GND-Pad4) -> GND
- J2 pad 1: unconnected-(J1-Pin_1-Pad1) -> +5V
- J2 pad 10: unconnected-(J1-Pin_10-Pad10) -> (no net)
- J2 pad 2: unconnected-(J1-Pin_2-Pad2) -> GND
- J2 pad 3: unconnected-(J1-Pin_3-Pad3) -> (no net)
- J2 pad 4: unconnected-(J1-Pin_4-Pad4) -> (no net)
- J2 pad 5: unconnected-(J1-Pin_5-Pad5) -> Net-(D4-A)
- J2 pad 6: unconnected-(J1-Pin_6-Pad6) -> (no net)
- J2 pad 7: unconnected-(J1-Pin_7-Pad7) -> (no net)
- J2 pad 8: unconnected-(J1-Pin_8-Pad8) -> (no net)
- J2 pad 9: unconnected-(J1-Pin_9-Pad9) -> (no net)
- R1 pad 2: unconnected-(R1-Pad2) -> Net-(D2-K)
- U1 pad 1: unconnected-(U1-~{RESET}/PB5-Pad1) -> Net-(J2-Pin_9)
- U1 pad 2: unconnected-(U1-XTAL1/PB3-Pad2) -> Net-(J2-Pin_7)
- U1 pad 3: unconnected-(U1-XTAL2/PB4-Pad3) -> Net-(J2-Pin_8)
- U1 pad 4: unconnected-(U1-GND-Pad4) -> GND
- U1 pad 5: unconnected-(U1-AREF/PB0-Pad5) -> Net-(J2-Pin_4)
- U1 pad 6: unconnected-(U1-PB1-Pad6) -> Net-(D4-A)
- U1 pad 7: unconnected-(U1-PB2-Pad7) -> Net-(J2-Pin_6)
- U1 pad 8: unconnected-(U1-VCC-Pad8) -> +5V
Other:
- board outline added: 45 x 45 mm
